File: zynq-test-board/power.kicad_sch (KiCad schematic)
At the start: 28 parts

Commit message: zynq-test-board: fix i2c addresses on power schematics
Other:
- note added: "= 0x40"
- note added: "= 0x41"
- note added: "= 0x42"
- note added: "= 0x43"
- note added: "= 0x44"
- note added: "= 0x45"
- note removed: "= 0x80"
- note removed: "= 0x82"
- note removed: "= 0x84"
- note removed: "= 0x86"
- note removed: "= 0x88"
- note removed: "= 0x8a"
Changed lines of the file:
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@@
     (stroke (width 0) (type default))
   )
-  (text "= 0x88" (at 233.68 92.71 0)
+  (text "= 0x44" (at 233.68 92.71 0)
     (effects (font (size 1.27 1.27)) (justify left bottom))
   )
-  (text "= 0x8a" (at 233.68 36.83 0)
+  (text "= 0x45" (at 233.68 36.83 0)
     (effects (font (size 1.27 1.27)) (justify left bottom))
   )
-  (text "= 0x82" (at 124.46 80.01 0)
+  (text "= 0x41" (at 124.46 80.01 0)
     (effects (font (size 1.27 1.27)) (justify left bottom))
   )
-  (text "= 0x80" (at 124.46 41.91 0)
+  (text "= 0x40" (at 124.46 41.91 0)
     (effects (font (size 1.27 1.27)) (justify left bottom))
   )
-  (text "= 0x86" (at 124.46 157.48 0)
+  (text "= 0x43" (at 124.46 157.48 0)
     (effects (font (size 1.27 1.27)) (justify left bottom))
   )
-  (text "= 0x84" (at 124.46 118.11 0)
+  (text "= 0x42" (at 124.46 118.11 0)
     (effects (font (size 1.27 1.27)) (justify left bottom))
   )
